File: PCB Kicad/transformerless-power-suply.kicad_pcb (KiCad board)
At the start: 2 copper layers, 18 parts, among them J1 Screw_Terminal_01x02, J2 Screw_Terminal_01x02, U1 LM7805_TO220

Commit message: Add files via upload
Parts:
- moved C3 97.2 mm to (172.5, 83.5), turned to 180 degrees
- moved J2 86.2 mm to (171.5, 93.0), turned to -90 degrees
- moved R2 82.2 mm to (153.5, 105.5), turned to 180 degrees
- moved R1 82.0 mm to (153.5, 100.0), turned to 180 degrees
- moved C2 78.2 mm to (149.5, 89.1), turned to -90 degrees
- moved U1 71.3 mm to (156.0, 76.0)
- moved D5 64.9 mm to (161.0, 83.5), turned to -90 degrees
- moved C1 64.7 mm to (148.0, 82.0)
- moved D6 64.7 mm to (161.0, 96.0), turned to -90 degrees
- moved R4 55.1 mm to (128.0, 99.5), turned to -90 degrees
- moved R3 54.3 mm to (124.5, 76.0), turned to -90 degrees
- moved D4 48.4 mm to (141.0, 96.0), turned to -90 degrees
- moved D1 47.5 mm to (134.0, 92.5), turned to 90 degrees
- moved D2 47.0 mm to (134.0, 96.0), turned to -90 degrees
- moved J1 46.3 mm to (124.0, 93.0), turned to 90 degrees
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Routing:
- net GNDREF: track 0.00 -> 129.6 mm
- net Net-(D1-K): track 0.00 -> 72.8 mm
- net Net-(D2-A): track 0.00 -> 32.3 mm
- net Net-(D1-A): track 0.00 -> 26.0 mm
- net Net-(J2-Pin_1): track 0.00 -> 24.4 mm
- net Net-(J1-Pin_2): track 0.00 -> 20.9 mm
- net Net-(D5-A): track 0.00 -> 18.7 mm
- net Net-(D6-A): track 0.00 -> 8.69 mm
- net Net-(D7-A): track 0.00 -> 6.67 mm
Other:
- board outline added: 61 x 42 mm
